Commit message: Restructured classes of the pathfinding
Same as before but:
-different structuring classes are more understandable and organised
-optimized scan data reading
-changes to data access and management

File: src/tea/urdf/tea.xacro (robot description, xacro)
@@ -27,5 +27,5 @@
   </joint>
   <joint name="hokuyo_joint" type="fixed">
-    <origin xyz="0.1 0 0.1" rpy="0 0 0" />
+    <origin xyz="0 0 0.12" rpy="0 0 0" />
     <parent link="chassis"/>
     <child link="hokuyo" />
@@ -141,5 +141,5 @@
   </link>
   <link name='chassis'>
-    <pose>0 0 0.1 0 0 0</pose>
+    <pose>0 0 0 0 0 0</pose>
     <inertial>
       <mass value="15.0"/>
